File: PCB/Projet_torero/capteur_bord_2.kicad_sch (KiCad schematic)
At the start: 0 parts

Commit message: ajout modif capteurs de bord
Parts:
- added QRD902: ~, Connector_JST:JST_EH_B4B-EH-A_1x04_P2.50mm_Vertical, symbol QRD1113:QRD1113
- added R901: 300R, symbol Device:R_Small
- added R902: 15.3k, symbol Device:R_Small
Connections:
- new net +5V: R901.1, R902.2
- new net ANALOG_OUTPUT_2: R902.1
Other:
- note added: "15.3k pour QRD1113 4.6k pour QRD1114"
- note added: "Anode"
- note added: "Cathode"
- note added: "Collector"
- note added: "Emitter"

Commit message: modif capteur
Connections:
- net ANALOG_OUTPUT_CAPT_BORD_2: now reaches R901.2
- net ANALOG_OUTPUT_2: no longer names the net of R902.1
Other:
- moved on the sheet: R901
Changed lines of the file:
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@@
 	(generator_version "8.0")
 	(paper "A4")
+	(junction
+		(at 69.85 107.95)
+		(diameter 0)
+		(color 0 0 0 0)
+	)
 	(wire
 		(pts
-			(xy 76.2 93.98) (xy 80.01 93.98)
+			(xy 69.85 106.68) (xy 69.85 107.95)
 		)
 		(stroke
@@
 		)
 	)
+	(wire
+		(pts
+			(xy 66.04 107.95) (xy 69.85 107.95)
+		)
+		(stroke
+			(width 0)
+			(type default)
+		)
+	)
+	(wire
+		(pts
+			(xy 69.85 107.95) (xy 69.85 110.49)
+		)
+		(stroke
+			(width 0)
+			(type default)
+		)
+	)
 	(text "Emitter"
 		(exclude_from_sim no)
@@
 	(text "Collector"
 		(exclude_from_sim no)
-		(at 64.008 114.3 0)
+		(at 64.008 118.11 0)
 		(effects
 			(font
@@
 		)
 	)
-	(hierarchical_label "ANALOG_OUTPUT_2"
+	(hierarchical_label "ANALOG_OUTPUT_CAPT_BORD_2"
 		(shape input)
-		(at 80.01 93.98 0)
+		(at 66.04 107.95 180)
 		(fields_autoplaced yes)
 		(effects
@@
 				(size 1.27 1.27)
 			)
-			(justify left)
+			(justify right)
 		)
 	)
 	(symbol
 		(lib_id "Device:R_Small")
-		(at 69.85 109.22 180)
+		(at 69.85 113.03 180)
 		(unit 1)
 		(exclude_from_sim no)
@@
 		(dnp no)
 		(property "Reference" "R901"
-			(at 64.77 109.22 90)
+			(at 64.77 113.03 90)
 			(effects
 				(font
@@
 		)
 		(property "Value" "300R"
-			(at 67.056 108.966 90)
+			(at 67.056 112.776 90)
 			(effects
 				(font
@@
 		)
 		(property "Footprint" ""
-			(at 69.85 109.22 0)
+			(at 69.85 113.03 0)
 			(effects
 				(font
@@
 		)
 		(property "Datasheet" "~"
-			(at 69.85 109.22 0)
+			(at 69.85 113.03 0)
 			(effects
 				(font
@@
 		)
 		(property "Description" "Resistor, small symbol"
-			(at 69.85 109.22 0)
+			(at 69.85 113.03 0)
 			(effects
 				(font
@@
 	(symbol
 		(lib_id "power:+5V")
-		(at 69.85 111.76 180)
+		(at 69.85 115.57 180)
 		(unit 1)
 		(exclude_from_sim no)
@@
 		(fields_autoplaced yes)
 		(property "Reference" "#PWR0901"
-			(at 69.85 107.95 0)
+			(at 69.85 111.76 0)
 			(effects
 				(font
@@
 		)
 		(property "Value" "+5V"
-			(at 69.8499 115.57 90)
+			(at 69.8499 119.38 90)
 			(effects
 				(font
@@
 		)
 		(property "Footprint" ""
-			(at 69.85 111.76 0)
+			(at 69.85 115.57 0)
 			(effects
 				(font
@@
 		)
 		(property "Datasheet" ""
-			(at 69.85 111.76 0)
+			(at 69.85 115.57 0)
 			(effects
 				(font
@@
 		)
 		(property "Description" "Power symbol creates a global label with name \"+5V\""
-			(at 69.85 111.76 0)
-			(effects
-				(font
+			(at 69.85 115.57 0)
+			(effects
+				(font

Commit message: review sch
Parts:
- R901: value 300R -> 300
- R902: value 15.3k -> 15k3
Connections:
- net ANALOG_OUTPUT_CAPT_BORD_2 renamed ANALOG_OUTPUT_CAPT_BORD_D
Changed lines of the file:
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@@
 		)
 	)
-	(hierarchical_label "ANALOG_OUTPUT_CAPT_BORD_2"
+	(hierarchical_label "ANALOG_OUTPUT_CAPT_BORD_D"
 		(shape input)
 		(at 66.04 107.95 180)
@@
 			)
 		)
-		(property "Value" "300R"
+		(property "Value" "300"
 			(at 67.056 112.776 90)
 			(effects
@@
 			)
 		)
-		(property "Value" "15.3k"
+		(property "Value" "15k3"
 			(at 78.74 87.376 90)
 			(effects
