File: PCB/Projet_torero/carpteur_bord_1.kicad_sch (KiCad schematic)
At the start: 0 parts

Commit message: ajout modif capteurs de bord
Parts:
- added QRD801: ~, Connector_JST:JST_EH_B4B-EH-A_1x04_P2.50mm_Vertical, symbol QRD1113:QRD1113
- added R803: 300R, symbol Device:R_Small
- added R804: 15.3k, symbol Device:R_Small
Connections:
- new net +5V: R803.1, R804.2
- new net ANALOG_OUTPUT_2: R804.1
Other:
- note added: "15.3k pour QRD1113 4.6k pour QRD1114"
- note added: "Anode"
- note added: "Cathode"
- note added: "Collector"
- note added: "Emitter"

Commit message: modif capteur
Connections:
- net ANALOG_OUTPUT_CAPT_BORD_1: now reaches R803.2
- net ANALOG_OUTPUT_2: no longer names the net of R804.1
Other:
- moved on the sheet: R803
Changed lines of the file:
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@@
 	(wire
 		(pts
-			(xy 69.85 52.07) (xy 73.66 52.07)
+			(xy 69.85 49.53) (xy 69.85 52.07)
 		)
 		(stroke
@@
 	(wire
 		(pts
-			(xy 69.85 49.53) (xy 69.85 52.07)
+			(xy 58.42 64.77) (xy 63.5 64.77)
 		)
 		(stroke
@@
 		)
 	)
+	(wire
+		(pts
+			(xy 63.5 68.58) (xy 63.5 64.77)
+		)
+		(stroke
+			(width 0)
+			(type default)
+		)
+	)
 	(text "15.3k pour QRD1113\n4.6k pour QRD1114\n"
 		(exclude_from_sim no)
@@
 	(text "Collector"
 		(exclude_from_sim no)
-		(at 57.658 72.39 0)
-		(effects
-			(font
-				(size 1.27 1.27)
-			)
-		)
-	)
-	(hierarchical_label "ANALOG_OUTPUT_2"
+		(at 57.658 76.2 0)
+		(effects
+			(font
+				(size 1.27 1.27)
+			)
+		)
+	)
+	(hierarchical_label "ANALOG_OUTPUT_CAPT_BORD_1"
 		(shape input)
-		(at 73.66 52.07 0)
+		(at 58.42 64.77 180)
 		(fields_autoplaced yes)
 		(effects
@@
 				(size 1.27 1.27)
 			)
-			(justify left)
+			(justify right)
 		)
 	)
 	(symbol
 		(lib_id "Device:R_Small")
-		(at 63.5 67.31 180)
+		(at 63.5 71.12 180)
 		(unit 1)
 		(exclude_from_sim no)
@@
 		(dnp no)
 		(property "Reference" "R803"
-			(at 58.42 67.31 90)
+			(at 58.42 71.12 90)
 			(effects
 				(font
@@
 		)
 		(property "Value" "300R"
-			(at 60.706 67.056 90)
+			(at 60.706 70.866 90)
 			(effects
 				(font
@@
 		)
 		(property "Footprint" ""
-			(at 63.5 67.31 0)
+			(at 63.5 71.12 0)
 			(effects
 				(font
@@
 		)
 		(property "Datasheet" "~"
-			(at 63.5 67.31 0)
+			(at 63.5 71.12 0)
 			(effects
 				(font
@@
 		)
 		(property "Description" "Resistor, small symbol"
-			(at 63.5 67.31 0)
+			(at 63.5 71.12 0)
 			(effects
 				(font
@@
 	(symbol
 		(lib_id "power:+5V")
-		(at 63.5 69.85 180)
+		(at 63.5 73.66 180)
 		(unit 1)
 		(exclude_from_sim no)
@@
 		(fields_autoplaced yes)
 		(property "Reference" "#PWR0806"
-			(at 63.5 66.04 0)
+			(at 63.5 69.85 0)
 			(effects
 				(font
@@
 		)
 		(property "Value" "+5V"
-			(at 63.4999 73.66 90)
+			(at 63.4999 77.47 90)
 			(effects
 				(font
@@
 		)
 		(property "Footprint" ""
-			(at 63.5 69.85 0)
+			(at 63.5 73.66 0)
 			(effects
 				(font
@@
 		)
 		(property "Datasheet" ""
-			(at 63.5 69.85 0)
+			(at 63.5 73.66 0)
 			(effects
 				(font
@@
 		)
 		(property "Description" "Power symbol creates a global label with name \"+5V\""
-			(at 63.5 69.85 0)
-			(effects
-				(font
+			(at 63.5 73.66 0)
+			(effects
+				(font

Commit message: review sch
Parts:
- R803: value 300R -> 300
- R804: value 15.3k -> 15k3
Connections:
- net ANALOG_OUTPUT_CAPT_BORD_1 renamed ANALOG_OUTPUT_CAPT_BORD_G
Changed lines of the file:
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@@
 		)
 	)
-	(hierarchical_label "ANALOG_OUTPUT_CAPT_BORD_1"
+	(hierarchical_label "ANALOG_OUTPUT_CAPT_BORD_G"
 		(shape input)
 		(at 58.42 64.77 180)
@@
 			)
 		)
-		(property "Value" "300R"
+		(property "Value" "300"
 			(at 60.706 70.866 90)
 			(effects
@@
 			)
 		)
-		(property "Value" "15.3k"
+		(property "Value" "15k3"
 			(at 72.39 45.466 90)
 			(effects

Commit message: review sch après vérif prof
Parts:
- removed QRD801: ~, Connector_JST:JST_EH_B4B-EH-A_1x04_P2.50mm_Vertical, symbol QRD1113:QRD1113
- removed R803: 300, symbol Device:R_Small
- removed R804: 15k3, symbol Device:R_Small
Other:
- note removed: "15.3k pour QRD1113 4.6k pour QRD1114"
- note removed: "Anode"
- note removed: "Cathode"
- note removed: "Collector"
- note removed: "Emitter"
