File: PCB/Projet_torero/CAPTEURS.kicad_sch (KiCad schematic)
At the start: 4 parts, among them J401 Conn_01x08, U401 ADXL343

Commit message: ajout valeur capa accelerometer
Parts:
- C401: value C_Small -> 1u
- C402: value C_Small -> 0.1u
Changed lines of the file:
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@@
 			)
 		)
-		(property "Value" "C_Small"
+		(property "Value" "1u"
 			(at 62.484 31.75 90)
 			(effects
@@
 			)
 		)
-		(property "Value" "C_Small"
+		(property "Value" "0.1u"
 			(at 67.564 45.974 90)
 			(effects

Commit message: modif capteur
Other:
- sheet Capteur de bord 1 ports: added ANALOG_OUTPUT_CAPT_BORD_1; removed none
- sheet Capteur de bord 2 ports: added ANALOG_OUTPUT_CAPT_BORD_2; removed none
Changed lines of the file:
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@@
+			)
+		)
+		(pin "ANALOG_OUTPUT_CAPT_BORD_2" input
+			(at 226.06 57.15 180)
+			(effects
+				(font
+					(size 1.27 1.27)
+				)
+				(justify left)
 			)
 		)
@@
 			)
 		)
+		(pin "ANALOG_OUTPUT_CAPT_BORD_1" input
+			(at 170.18 57.15 180)
+			(effects
+				(font
+					(size 1.27 1.27)
+				)
+				(justify left)
+			)
+		)

Commit message: review sch
Parts:
- C402: value 0.1u -> 100n
Connections:
- net CS renamed CS_ACC
- net DEV_EN renamed DEV_EN_LIDAR
- net INT1 renamed INT1_ACC
- net INT2 renamed INT2_ACC
- net M_EN renamed M_EN_LIDAR
- net M_SCTR renamed M_SCTR_LIDAR
- net Rx renamed Rx_LIDAR
- net SCLK renamed SCLK_ACC
- net SDA/SDI/SDIO renamed SDI_ACC
- net SDO/ADDR renamed SDO_ACC
- net Tx renamed Tx_LIDAR
Other:
- sheet Capteur de bord 1 renamed Capteur de bord G
- sheet Capteur de bord 2 renamed Capteur de bord D
- sheet Capteur de bord D ports: added ANALOG_OUTPUT_CAPT_BORD_D; removed ANALOG_OUTPUT_CAPT_BORD_2
- sheet Capteur de bord G ports: added ANALOG_OUTPUT_CAPT_BORD_G; removed ANALOG_OUTPUT_CAPT_BORD_1
- note added: "CAPTEUR BORDURE DROITE"
- note added: "CAPTEUR BORDURE GAUCHE"
- note removed: "CAPTEUR BORDURE"
Changed lines of the file:
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@@
 	(polyline
 		(pts
-			(xy 107.95 99.06) (xy 107.95 198.12)
+			(xy 162.56 195.58) (xy 162.56 198.12)
 		)
 		(stroke
@@
 	(wire
 		(pts
+			(xy 214.63 137.16) (xy 223.52 137.16)
+		)
+		(stroke
+			(width 0)
+			(type default)
+		)
+	)
+	(wire
+		(pts
 			(xy 58.42 48.26) (xy 58.42 50.8)
 		)
@@
 		)
 	)
+	(polyline
+		(pts
+			(xy 162.56 99.06) (xy 162.56 198.12)
+		)
+		(stroke
+			(width 0)
+			(type default)
+		)
+	)
 	(wire
 		(pts
-			(xy 128.27 54.61) (xy 134.62 54.61)
+			(xy 215.9 62.23) (xy 223.52 62.23)
+		)
+		(stroke
+			(width 0)
+			(type default)
+		)
+	)
+	(wire
+		(pts
+			(xy 121.92 54.61) (xy 134.62 54.61)
 		)
 		(stroke
@@
 		)
 	)
+	(text "CAPTEUR BORDURE DROITE\n"
+		(exclude_from_sim no)
+		(at 198.882 107.95 0)
+		(effects
+			(font
+				(size 2 2)
+			)
+		)
+	)
 	(text "ACCELEROMETER"
 		(exclude_from_sim no)
@@
 		)
 	)
-	(text "CAPTEUR BORDURE"
+	(text "CAPTEUR BORDURE GAUCHE\n"
 		(exclude_from_sim no)
 		(at 198.374 19.812 0)
@@
 		)
 	)
-	(hierarchical_label "Tx"
+	(hierarchical_label "ANALOG_OUTPUT_CAPT_BORD_G"
+		(shape input)
+		(at 215.9 62.23 180)
+		(fields_autoplaced yes)
+		(effects
+			(font
+				(size 1.27 1.27)
+			)
+			(justify right)
+		)
+	)
+	(hierarchical_label "Tx_LIDAR"
 		(shape input)
 		(at 134.62 59.69 180)
@@
 		)
 	)
-	(hierarchical_label "M_SCTR"
+	(hierarchical_label "M_SCTR_LIDAR"
 		(shape input)
 		(at 134.62 52.07 180)
@@
 		)
 	)
-	(hierarchical_label "SDO{slash}ADDR"
+	(hierarchical_label "SDO_ACC"
 		(shape input)
 		(at 45.72 60.96 180)
@@
 		)
 	)
-	(hierarchical_label "M_EN"
+	(hierarchical_label "M_EN_LIDAR"
 		(shape input)
 		(at 134.62 46.99 180)
@@
 		)
 	)
-	(hierarchical_label "DEV_EN"
+	(hierarchical_label "DEV_EN_LIDAR"
 		(shape input)
 		(at 134.62 49.53 180)
@@
 		)
 	)
-	(hierarchical_label "INT1"
+	(hierarchical_label "INT1_ACC"
 		(shape input)
 		(at 71.12 63.5 0)
@@
 		)
 	)
-	(hierarchical_label "CS"
+	(hierarchical_label "CS_ACC"
 		(shape input)
 		(at 45.72 68.58 180)
@@
 		)
 	)
-	(hierarchical_label "INT2"
+	(hierarchical_label "INT2_ACC"
 		(shape input)
 		(at 71.12 66.04 0)
@@
 		)
 	)
-	(hierarchical_label "SDA{slash}SDI{slash}SDIO"
+	(hierarchical_label "SDI_ACC"
 		(shape input)
 		(at 45.72 63.5 180)
@@
 		)
 	)
-	(hierarchical_label "SCLK"
+	(hierarchical_label "SCLK_ACC"
 		(shape input)
 		(at 45.72 66.04 180)
@@
 		)
 	)
-	(hierarchical_label "Rx"
+	(hierarchical_label "Rx_LIDAR"
 		(shape input)
 		(at 134.62 57.15 180)
+		(fields_autoplaced yes)
+		(effects
+			(font
+				(size 1.27 1.27)
+			)
+			(justify right)
+		)
+	)
+	(hierarchical_label "ANALOG_OUTPUT_CAPT_BORD_D"
+		(shape input)
+		(at 214.63 137.16 180)
 		(fields_autoplaced yes)
 		(effects
@@
 	(symbol
 		(lib_id "power:GND")
-		(at 128.27 54.61 0)
+		(at 121.92 54.61 0)
 		(unit 1)
 		(exclude_from_sim no)
@@
 		(fields_autoplaced yes)
 		(property "Reference" "#PWR0406"
-			(at 128.27 60.96 0)
+			(at 121.92 60.96 0)
 			(effects
 				(font
@@
 		)
 		(property "Value" "GND"
-			(at 128.27 59.69 0)
+			(at 121.92 59.69 0)
 			(effects
 				(font
@@
 		)
 		(property "Footprint" ""
-			(at 128.27 54.61 0)
+			(at 121.92 54.61 0)
 			(effects
 				(font
@@
 		)
 		(property "Datasheet" ""
-			(at 128.27 54.61 0)
+			(at 121.92 54.61 0)
 			(effects
 				(font
@@
 		)
 		(property "Description" "Power symbol creates a global label with name \"GND\" , ground"
-			(at 128.27 54.61 0)
+			(at 121.92 54.61 0)
 			(effects
 				(font
@@
 			)
 		)
-		(property "Value" "0.1u"
+		(property "Value" "100n"
 			(at 67.564 45.974 90)
 			(effects
@@
 	)
 	(sheet
-		(at 226.06 39.37)
+		(at 223.52 119.38)
 		(size 48.26 36.83)
 		(fields_autoplaced yes)
@@
 			(color 0 0 0 0.0000)
 		)
-		(property "Sheetname" "Capteur de bord 2"
-			(at 226.06 38.6584 0)
+		(property "Sheetname" "Capteur de bord D"
+			(at 223.52 118.6684 0)
 			(effects
 				(font
@@
 		)
 		(property "Sheetfile" "capteur_bord_2.kicad_sch"
-			(at 226.06 76.7846 0)
+			(at 223.52 156.7946 0)
 			(effects
 				(font
@@
 			)
 		)
-		(pin "ANALOG_OUTPUT_CAPT_BORD_2" input
-			(at 226.06 57.15 180)
+		(pin "ANALOG_OUTPUT_CAPT_BORD_D" input
+			(at 223.52 137.16 180)
 			(effects
 				(font
@@
 	)
 	(sheet
-		(at 170.18 39.37)
+		(at 223.52 44.45)
 		(size 46.99 36.83)
 		(fields_autoplaced yes)
@@
 			(color 0 0 0 0.0000)
 		)
-		(property "Sheetname" "Capteur de bord 1"
-			(at 170.18 38.6584 0)
+		(property "Sheetname" "Capteur de bord G"
+			(at 223.52 43.7384 0)
 			(effects
 				(font
@@
 		)
 		(property "Sheetfile" "carpteur_bord_1.kicad_sch"
-			(at 170.18 76.7846 0)
+			(at 223.52 81.8646 0)
 			(effects
 				(font
@@
 			)
 		)
-		(pin "ANALOG_OUTPUT_CAPT_BORD_1" input
-			(at 170.18 57.15 180)
-			(effects
-				(font
+		(pin "ANALOG_OUTPUT_CAPT_BORD_G" input
+			(at 223.52 62.23 180)
+			(effects
+				(font

Commit message: review sch après vérif prof
Connections:
- net +3.3VA is gone; now on net +3.3V: C402.1, U401.1 (Vdd_I/O)
- net +3.3V: no longer U401.3 (RES)
- no-connect marks 1 -> 2
Other:
- sheet Capteur de bord D: file capteur_bord_2.kicad_sch -> Capteur_Bord.kicad_sch
- sheet Capteur de bord D ports: added ANALOG_OUTPUT_CAPT_BORD; removed ANALOG_OUTPUT_CAPT_BORD_D
- sheet Capteur de bord G: file carpteur_bord_1.kicad_sch -> Capteur_Bord.kicad_sch
- sheet Capteur de bord G ports: added ANALOG_OUTPUT_CAPT_BORD; removed ANALOG_OUTPUT_CAPT_BORD_G
Changed lines of the file:
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@@
-	)
-	(junction
-		(at 58.42 48.26)
-		(diameter 0)
-		(color 0 0 0 0)
 	)
 	(junction
@@
 		(at 134.62 44.45)
 	)
+	(no_connect
+		(at 53.34 50.8)
+	)
 	(polyline
 		(pts
@@
 	(wire
 		(pts
-			(xy 58.42 48.26) (xy 58.42 50.8)
+			(xy 58.42 35.56) (xy 58.42 50.8)
+		)
+		(stroke
+			(width 0)
+			(type default)
+		)
+	)
+	(polyline
+		(pts
+			(xy 162.56 99.06) (xy 162.56 198.12)
 		)
 		(stroke
@@
 	(wire
 		(pts
-			(xy 58.42 35.56) (xy 58.42 48.26)
+			(xy 215.9 62.23) (xy 223.52 62.23)
+		)
+		(stroke
+			(width 0)
+			(type default)
+		)
+	)
+	(wire
+		(pts
+			(xy 121.92 54.61) (xy 134.62 54.61)
 		)
 		(stroke
@@
 	(polyline
 		(pts
-			(xy 162.56 99.06) (xy 162.56 198.12)
+			(xy 107.95 12.7) (xy 107.95 99.06)
+		)
+		(stroke
+			(width 0)
+			(type default)
+		)
+	)
+	(polyline
+		(pts
+			(xy 162.56 12.7) (xy 162.56 99.06)
+		)
+		(stroke
+			(width 0)
+			(type default)
+		)
+	)
+	(polyline
+		(pts
+			(xy 13.97 99.06) (xy 284.48 99.06)
 		)
 		(stroke
@@
 	(wire
 		(pts
-			(xy 215.9 62.23) (xy 223.52 62.23)
+			(xy 63.5 49.53) (xy 63.5 50.8)
 		)
 		(stroke
@@
 	(wire
 		(pts
-			(xy 121.92 54.61) (xy 134.62 54.61)
-		)
-		(stroke
-			(width 0)
-			(type default)
-		)
-	)
-	(polyline
-		(pts
-			(xy 107.95 12.7) (xy 107.95 99.06)
-		)
-		(stroke
-			(width 0)
-			(type default)
-		)
-	)
-	(polyline
-		(pts
-			(xy 162.56 12.7) (xy 162.56 99.06)
-		)
-		(stroke
-			(width 0)
-			(type default)
-		)
-	)
-	(polyline
-		(pts
-			(xy 13.97 99.06) (xy 284.48 99.06)
-		)
-		(stroke
-			(width 0)
-			(type default)
-		)
-	)
-	(wire
-		(pts
-			(xy 63.5 49.53) (xy 63.5 50.8)
-		)
-		(stroke
-			(width 0)
-			(type default)
-		)
-	)
-	(wire
-		(pts
 			(xy 63.5 45.72) (xy 63.5 49.53)
-		)
-		(stroke
-			(width 0)
-			(type default)
-		)
-	)
-	(wire
-		(pts
-			(xy 53.34 48.26) (xy 58.42 48.26)
-		)
-		(stroke
-			(width 0)
-			(type default)
-		)
-	)
-	(wire
-		(pts
-			(xy 53.34 50.8) (xy 53.34 48.26)
 		)
 		(stroke
@@
 	)
 	(symbol
+		(lib_id "power:+3.3V")
+		(at 63.5 45.72 0)
+		(unit 1)
+		(exclude_from_sim no)
+		(in_bom yes)
+		(on_board yes)
+		(dnp no)
+		(fields_autoplaced yes)
+		(property "Reference" "#PWR0403"
+			(at 63.5 49.53 0)
+			(effects
+				(font
+					(size 1.27 1.27)
+				)
+				(hide yes)
+			)
+		)
+		(property "Value" "+3.3V"
+			(at 63.5 40.64 0)
+			(effects
+				(font
+					(size 1.27 1.27)
+				)
+			)
+		)
+		(property "Footprint" ""
+			(at 63.5 45.72 0)
+			(effects
+				(font
+					(size 1.27 1.27)
+				)
+				(hide yes)
+			)
+		)
+		(property "Datasheet" ""
+			(at 63.5 45.72 0)
+			(effects
+				(font
+					(size 1.27 1.27)
+				)
+				(hide yes)
+			)
+		)
+		(property "Description" "Power symbol creates a global label with name \"+3.3V\""
+			(at 63.5 45.72 0)
+			(effects
+				(font
+					(size 1.27 1.27)
+				)
+				(hide yes)
+			)
+		)
+		(pin "1"
+		)
+		(instances
+			(project "Projet_torero"
+				(path "/04e1eb47-a2c4-462b-bef7-377d9515a2c0/15f7fbe2-20f5-4588-8b16-1e568ab2921c"
+					(reference "#PWR0403")
+					(unit 1)
+				)
+			)
+		)
+	)
+	(symbol
 		(lib_id "power:GND")
 		(at 58.42 76.2 0)
@@
 		(dnp no)
 		(property "Reference" "C402"
-			(at 66.0463 43.18 90)
+			(at 72.644 41.656 90)
 			(effects
 				(font
@@
 	)
 	(symbol
-		(lib_id "power:+3.3VA")
-		(at 63.5 45.72 0)
-		(unit 1)
-		(exclude_from_sim no)
-		(in_bom yes)
-		(on_board yes)
-		(dnp no)
-		(fields_autoplaced yes)
-		(property "Reference" "#PWR0403"
-			(at 63.5 49.53 0)
-			(effects
-				(font
-					(size 1.27 1.27)
-				)
-				(hide yes)
-			)
-		)
-		(property "Value" "+3.3VA"
-			(at 63.5 40.64 0)
-			(effects
-				(font
-					(size 1.27 1.27)
-				)
-			)
-		)
-		(property "Footprint" ""
-			(at 63.5 45.72 0)
-			(effects
-				(font
-					(size 1.27 1.27)
-				)
-				(hide yes)
-			)
-		)
-		(property "Datasheet" ""
-			(at 63.5 45.72 0)
-			(effects
-				(font
-					(size 1.27 1.27)
-				)
-				(hide yes)
-			)
-		)
-		(property "Description" "Power symbol creates a global label with name \"+3.3VA\""
-			(at 63.5 45.72 0)
-			(effects
-				(font
-					(size 1.27 1.27)
-				)
-				(hide yes)
-			)
-		)
-		(pin "1"
-		)
-		(instances
-			(project ""
-				(path "/04e1eb47-a2c4-462b-bef7-377d9515a2c0/15f7fbe2-20f5-4588-8b16-1e568ab2921c"
-					(reference "#PWR0403")
-					(unit 1)
-				)
-			)
-		)
-	)
-	(symbol
 		(lib_id "power:GND")
 		(at 63.5 35.56 90)
@@
 	(sheet
 		(at 223.52 119.38)
-		(size 48.26 36.83)
+		(size 46.99 36.83)
 		(fields_autoplaced yes)
 		(stroke
@@
 			)
 		)
-		(property "Sheetfile" "capteur_bord_2.kicad_sch"
+		(property "Sheetfile" "Capteur_Bord.kicad_sch"
 			(at 223.52 156.7946 0)
 			(effects
@@
 			)
 		)
-		(pin "ANALOG_OUTPUT_CAPT_BORD_D" input
+		(pin "ANALOG_OUTPUT_CAPT_BORD" input
 			(at 223.52 137.16 180)
 			(effects
@@
 			)
 		)
-		(property "Sheetfile" "carpteur_bord_1.kicad_sch"
+		(property "Sheetfile" "Capteur_Bord.kicad_sch"
 			(at 223.52 81.8646 0)
 			(effects
@@
 			)
 		)
-		(pin "ANALOG_OUTPUT_CAPT_BORD_G" input
+		(pin "ANALOG_OUTPUT_CAPT_BORD" input
 			(at 223.52 62.23 180)
 			(effects

Commit message: modif placement composant
Parts:
- C401: footprint (none) -> Capacitor_SMD:C_0603_1608Metric
- C402: footprint (none) -> Capacitor_SMD:C_0402_1005Metric
- J401: footprint (none) -> Connector_JST:JST_XH_S8B-XH-A_1x08_P2.50mm_Horizontal
Connections:
- net +3.3V: now also C402.2; no longer C402.1
- net GND: now also C402.1; no longer C402.2
Other:
- moved on the sheet: C402
Changed lines of the file:
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@@
+	)
+	(junction
+		(at 63.5 49.53)
+		(diameter 0)
+		(color 0 0 0 0)
 	)
 	(junction
@@
 		(color 0 0 0 0)
 	)
-	(junction
-		(at 63.5 49.53)
-		(diameter 0)
-		(color 0 0 0 0)
-	)
 	(no_connect
 		(at 134.62 44.45)
@@
 		)
 	)
+	(wire
+		(pts
+			(xy 63.5 49.53) (xy 63.5 50.8)
+		)
+		(stroke
+			(width 0)
+			(type default)
+		)
+	)
 	(polyline
 		(pts
@@
 		(pts
 			(xy 13.97 99.06) (xy 284.48 99.06)
-		)
-		(stroke
-			(width 0)
-			(type default)
-		)
-	)
-	(wire
-		(pts
-			(xy 63.5 49.53) (xy 63.5 50.8)
 		)
 		(stroke
@@
 			)
 		)
-		(property "Footprint" ""
+		(property "Footprint" "Capacitor_SMD:C_0603_1608Metric"
 			(at 60.96 35.56 0)
 			(effects
@@
 			)
 		)
-		(property "Footprint" ""
+		(property "Footprint" "Connector_JST:JST_XH_S8B-XH-A_1x08_P2.50mm_Horizontal"
 			(at 139.7 52.07 0)
 			(effects
@@
 	(symbol
 		(lib_id "Device:C_Small")
-		(at 66.04 49.53 90)
+		(at 66.04 49.53 270)
 		(unit 1)
 		(exclude_from_sim no)
@@
 		(dnp no)
 		(property "Reference" "C402"
-			(at 72.644 41.656 90)
+			(at 59.436 57.404 90)
 			(effects
 				(font
@@
 		)
 		(property "Value" "100n"
-			(at 67.564 45.974 90)
-			(effects
-				(font
-					(size 1.27 1.27)
-				)
-			)
-		)
-		(property "Footprint" ""
+			(at 64.516 53.086 90)
+			(effects
+				(font
+					(size 1.27 1.27)
+				)
+			)
+		)
+		(property "Footprint" "Capacitor_SMD:C_0402_1005Metric"
 			(at 66.04 49.53 0)
 			(effects
