File: PCB/Projet_torero/Projet_torero.kicad_pcb (KiCad board)
At the start: 4 copper layers, 54 x 57 mm, 75 parts, among them IC501 MP1475SGJ-P, J201 Conn_02x07_Odd_Even, J202 Conn_02x08_Odd_Even, J401 Conn_01x08, J501 Conn_01x02, J502 Conn_01x02, J601 Conn_01x06, J701 Conn_01x06, SW201 SW_Push, SW202 SW_Push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

Commit message: changement pin usart2
Connections:
- U201 pad 10: VCP_TX -> LED_E
- U201 pad 11: VCP_RX -> /CAPTEURS/DEV_EN_LIDAR
- U201 pad 38: /CAPTEURS/DEV_EN_LIDAR -> VCP_RX
- U201 pad 40: STATUS_LED_Debug -> VCP_TX
- U201 pad 44: LED_E -> STATUS_LED_Debug
Changed lines of the file:
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@@
 		(tags "resistor")
 		(property "Reference" "R202"
-			(at 0 -1.43 360)
+			(at 0 -1.43 0)
 			(layer "F.SilkS")
 			(effects
@@
 		)
 		(property "Value" "120"
-			(at 0 1.43 360)
+			(at 0 1.43 0)
 			(layer "F.Fab")
 			(effects
@@
 		)
 		(fp_text user "${REFERENCE}"
-			(at 0 0 360)
+			(at 0 0 0)
 			(layer "F.Fab")
 			(effects
@@
 		(tags "LED handsolder")
 		(property "Reference" "D201"
-			(at 0 -1.43 360)
+			(at 0 -1.43 0)
 			(layer "F.SilkS")
 			(effects
@@
 		)
 		(property "Value" "Green"
-			(at 0 1.43 360)
+			(at 0 1.43 0)
 			(layer "F.Fab")
 			(effects
@@
 		)
 		(fp_text user "${REFERENCE}"
-			(at 0 0 360)
+			(at 0 0 0)
 			(layer "F.Fab")
 			(effects
@@
 		(tags "capacitor")
 		(property "Reference" "C703"
-			(at -0.125 -1.475 360)
+			(at -0.125 -1.475 0)
 			(layer "F.SilkS")
 			(effects
@@
 		)
 		(property "Value" "1u"
-			(at 0 1.43 360)
+			(at 0 1.43 0)
 			(layer "F.Fab")
 			(effects
@@
 		)
 		(fp_text user "${REFERENCE}"
-			(at 0 0 360)
+			(at 0 0 0)
 			(layer "F.Fab")
 			(effects
@@
 		(tags "resistor")
 		(property "Reference" "R204"
-			(at -1.38 -11.81 360)
+			(at -1.38 -11.81 0)
 			(layer "F.SilkS")
 			(effects
@@
 		)
 		(fp_text user "${REFERENCE}"
-			(at 0 0 360)
+			(at 0 0 0)
 			(layer "F.Fab")
 			(effects
@@
 		(tags "Integrated Circuit")
 		(property "Reference" "IC501"
-			(at 0 0 360)
+			(at 0 0 0)
 			(layer "F.SilkS")
 			(effects
@@
 			(layers "F.Cu" "F.Paste" "F.Mask")
 			(roundrect_rratio 0.25)
-			(net 49 "VCP_TX")
+			(net 51 "LED_E")
 			(pinfunction "PA2")
 			(pintype "bidirectional")
@@
 			(layers "F.Cu" "F.Paste" "F.Mask")
 			(roundrect_rratio 0.25)
-			(net 48 "VCP_RX")
+			(net 34 "/CAPTEURS/DEV_EN_LIDAR")
 			(pinfunction "PA3")
 			(pintype "bidirectional")
@@
 			(layers "F.Cu" "F.Paste" "F.Mask")
 			(roundrect_rratio 0.25)
-			(net 34 "/CAPTEURS/DEV_EN_LIDAR")
+			(net 48 "VCP_RX")
 			(pinfunction "PA15")
 			(pintype "bidirectional")
@@
 			(layers "F.Cu" "F.Paste" "F.Mask")
 			(roundrect_rratio 0.25)
-			(net 81 "STATUS_LED_Debug")
+			(net 49 "VCP_TX")
 			(pinfunction "PC11")
 			(pintype "bidirectional")
@@
 			(layers "F.Cu" "F.Paste" "F.Mask")
 			(roundrect_rratio 0.25)
-			(net 51 "LED_E")
+			(net 81 "STATUS_LED_Debug")
 			(pinfunction "PB6")
 			(pintype "bidirectional")
@@
 		(tags "resistor")
 		(property "Reference" "10k201"
-			(at 0 -1.43 360)
+			(at 0 -1.43 0)
 			(layer "F.SilkS")
 			(effects
@@
 		)
 		(property "Value" "10k"
-			(at 0 1.43 360)
+			(at 0 1.43 0)
 			(layer "F.Fab")
 			(effects
@@
 		)
 		(fp_text user "${REFERENCE}"
-			(at 0 0 360)
+			(at 0 0 0)
 			(layer "F.Fab")
 			(effects
@@
 		(tags "capacitor")
 		(property "Reference" "C504"
-			(at 0 -1.43 360)
+			(at 0 -1.43 0)
 			(layer "F.SilkS")
 			(effects
@@
 		)
 		(property "Value" "47u"
-			(at 0 1.43 360)
+			(at 0 1.43 0)
 			(layer "F.Fab")
 			(effects
@@
 		)
 		(fp_text user "${REFERENCE}"
-			(at 0 0 360)
+			(at 0 0 0)
 			(layer "F.Fab")
 			(effects
@@
 		(tags "capacitor")
 		(property "Reference" "C501"
-			(at 0 0 360)
+			(at 0 0 0)
 			(layer "F.SilkS")
 			(effects
@@
 		)
 		(property "Value" "22u"
-			(at 0 1.68 360)
+			(at 0 1.68 0)
 			(layer "F.Fab")
 			(effects
@@
 		)
 		(fp_text user "${REFERENCE}"
-			(at 0 0 360)
+			(at 0 0 0)
 			(layer "F.Fab")
 			(effects
@@
 		(tags "capacitor")
 		(property "Reference" "C603"
-			(at 0 -1.43 360)
+			(at 0 -1.43 0)
 			(layer "F.SilkS")
 			(effects
@@
 		)
 		(property "Value" "1u"
-			(at 0 1.43 360)
+			(at 0 1.43 0)
 			(layer "F.Fab")
 			(effects
@@
 		)
 		(fp_text user "${REFERENCE}"
-			(at 0 0 360)
+			(at 0 0 0)
 			(layer "F.Fab")
 			(effects
@@
 		(tags "resistor")
 		(property "Reference" "R501"
-			(at 0 0 360)
+			(at 0 0 0)
 			(layer "F.SilkS")
 			(effects
@@
 		)
 		(property "Value" "100k"
-			(at 0 1.43 360)
+			(at 0 1.43 0)
 			(layer "F.Fab")
 			(effects
@@
 		)
 		(fp_text user "${REFERENCE}"
-			(at 0 0 360)
+			(at 0 0 0)
 			(layer "F.Fab")
 			(effects
@@
 		(tags "capacitor")
 		(property "Reference" "C503"
-			(at 0.25 -1.375 360)
+			(at 0.25 -1.375 0)
 			(layer "F.SilkS")
 			(effects
@@
 		)
 		(property "Value" "100n"
-			(at 0 1.16 360)
+			(at 0 1.16 0)
 			(layer "F.Fab")
 			(effects
@@
 		)
 		(fp_text user "${REFERENCE}"
-			(at 0 0 360)
+			(at 0 0 0)
 			(layer "F.Fab")
 			(effects
@@
 		(tags "Surface mounted pin header SMD 2x07 1.27mm double row")
 		(property "Reference" "J201"
-			(at -0.05 -5.76 360)
+			(at -0.05 -5.76 0)
 			(layer "F.SilkS")
 			(effects
@@
 		)
 		(property "Value" "Conn_02x07_Odd_Even"
-			(at 0 5.505 360)
+			(at 0 5.505 0)
 			(layer "F.Fab")
 			(hide yes)
@@
 		(tags "capacitor")
 		(property "Reference" "C401"
-			(at 0.025 -1.35 360)
+			(at 0.025 -1.35 0)
 			(layer "F.SilkS")
 			(effects
@@
 		)
 		(property "Value" "1u"
-			(at 0 1.43 360)
+			(at 0 1.43 0)
 			(layer "F.Fab")
 			(effects
@@
 		)
 		(fp_text user "${REFERENCE}"
-			(at 0 0 360)
+			(at 0 0 0)
 			(layer "F.Fab")
 			(effects
@@
 		(tags "capacitor")
 		(property "Reference" "C205"
-			(at 0 -1.43 360)
+			(at 0 -1.43 0)
 			(layer "F.SilkS")
 			(effects
@@
 		)
 		(property "Value" "1u"
-			(at 0 1.43 360)
+			(at 0 1.43 0)
 			(layer "F.Fab")
 			(effects
@@
 		)
 		(fp_text user "${REFERENCE}"
-			(at 0 0 360)
+			(at 0 0 0)
 			(layer "F.Fab")
 			(effects
@@
 		(tags "resistor")
 		(property "Reference" "R502"
-			(at 0 0 360)
+			(at 0 0 0)
 			(layer "F.SilkS")
 			(effects
@@
 		)
 		(property "Value" "100k"
-			(at 0 1.43 360)
+			(at 0 1.43 0)
 			(layer "F.Fab")
 			(effects
@@
 		)
 		(fp_text user "${REFERENCE}"
-			(at 0 0 360)
+			(at 0 0 0)
 			(layer "F.Fab")
 			(effects
@@
 		)
 		(fp_text user "${REFERENCE}"
-			(at 0 0 360)
+			(at 0 0 0)
 			(layer "F.Fab")
 			(effects
@@
 		(tags "capacitor")
 		(property "Reference" "C402"
-			(at 0 -1.16 360)
+			(at 0 -1.16 0)
 			(layer "F.SilkS")
 			(effects
@@
 		)
 		(property "Value" "100n"
-			(at 0 1.16 360)
+			(at 0 1.16 0)
 			(layer "F.Fab")
 			(effects
@@
 		)
 		(fp_text user "${REFERENCE}"
-			(at 0 0 360)
+			(at 0 0 0)
 			(layer "F.Fab")
 			(effects

Commit message: rectification erreur pin usart2
Connections:
- U201 pad 10: LED_E -> VCP_TX
- U201 pad 11: /CAPTEURS/DEV_EN_LIDAR -> VCP_RX
- U201 pad 38: VCP_RX -> /CAPTEURS/DEV_EN_LIDAR
- U201 pad 40: VCP_TX -> STATUS_LED_Debug
- U201 pad 44: STATUS_LED_Debug -> LED_E
Changed lines of the file:
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@@
 			(layers "F.Cu" "F.Paste" "F.Mask")
 			(roundrect_rratio 0.25)
-			(net 51 "LED_E")
+			(net 49 "VCP_TX")
 			(pinfunction "PA2")
 			(pintype "bidirectional")
@@
 			(layers "F.Cu" "F.Paste" "F.Mask")
 			(roundrect_rratio 0.25)
-			(net 34 "/CAPTEURS/DEV_EN_LIDAR")
+			(net 48 "VCP_RX")
 			(pinfunction "PA3")
 			(pintype "bidirectional")
@@
 			(layers "F.Cu" "F.Paste" "F.Mask")
 			(roundrect_rratio 0.25)
-			(net 48 "VCP_RX")
+			(net 34 "/CAPTEURS/DEV_EN_LIDAR")
 			(pinfunction "PA15")
 			(pintype "bidirectional")
@@
 			(layers "F.Cu" "F.Paste" "F.Mask")
 			(roundrect_rratio 0.25)
-			(net 49 "VCP_TX")
+			(net 81 "STATUS_LED_Debug")
 			(pinfunction "PC11")
 			(pintype "bidirectional")
@@
 			(layers "F.Cu" "F.Paste" "F.Mask")
 			(roundrect_rratio 0.25)
-			(net 81 "STATUS_LED_Debug")
+			(net 51 "LED_E")
 			(pinfunction "PB6")
 			(pintype "bidirectional")
