File: PCB/Projet_torero/Moteur.kicad_sch (KiCad schematic)
At the start: 5 parts, among them J602 Conn_01x06, U601 ZXBM5210-SP

Commit message: modif capa moteur
Parts:
- C603: value 1µF -> 1u
Changed lines of the file:
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@@
 			)
 		)
-		(property "Value" "1µF"
+		(property "Value" "1u"
 			(at 155.956 67.564 90)
 			(effects

Commit message: review sch après vérif prof
Other:
- moved on the sheet: C603
Changed lines of the file:
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@@
+	)
+	(junction
+		(at 167.64 63.5)
+		(diameter 0)
+		(color 0 0 0 0)
 	)
 	(junction
@@
 	)
 	(junction
-		(at 162.56 63.5)
-		(diameter 0)
-		(color 0 0 0 0)
-	)
-	(junction
 		(at 137.16 45.72)
 		(diameter 0)
@@
 	(wire
 		(pts
+			(xy 162.56 69.85) (xy 162.56 71.12)
+		)
+		(stroke
+			(width 0)
+			(type default)
+		)
+	)
+	(wire
+		(pts
 			(xy 137.16 39.37) (xy 142.24 39.37)
 		)
@@
 	(wire
 		(pts
-			(xy 162.56 63.5) (xy 185.42 63.5)
-		)
-		(stroke
-			(width 0)
-			(type default)
-		)
-	)
-	(wire
-		(pts
-			(xy 162.56 69.85) (xy 162.56 71.12)
+			(xy 162.56 63.5) (xy 167.64 63.5)
 		)
 		(stroke
@@
 	(wire
 		(pts
-			(xy 162.56 63.5) (xy 162.56 64.77)
+			(xy 167.64 63.5) (xy 167.64 64.77)
 		)
 		(stroke
@@
 		(pts
 			(xy 149.86 73.66) (xy 185.42 73.66)
+		)
+		(stroke
+			(width 0)
+			(type default)
+		)
+	)
+	(wire
+		(pts
+			(xy 167.64 63.5) (xy 185.42 63.5)
+		)
+		(stroke
+			(width 0)
+			(type default)
+		)
+	)
+	(wire
+		(pts
+			(xy 167.64 69.85) (xy 162.56 69.85)
 		)
 		(stroke
@@
 	(symbol
 		(lib_id "Device:C_Small")
-		(at 162.56 67.31 0)
+		(at 167.64 67.31 0)
 		(unit 1)
 		(exclude_from_sim no)
@@
 		(dnp no)
 		(property "Reference" "C603"
-			(at 158.496 67.564 90)
+			(at 163.576 67.564 90)
 			(effects
 				(font
@@
 		)
 		(property "Value" "1u"
-			(at 155.956 67.564 90)
+			(at 161.036 67.564 90)
 			(effects
 				(font
@@
 		)
 		(property "Footprint" ""
-			(at 162.56 67.31 0)
+			(at 167.64 67.31 0)
 			(effects
 				(font
@@
 		)
 		(property "Datasheet" "~"
-			(at 162.56 67.31 0)
+			(at 167.64 67.31 0)
 			(effects
 				(font
@@
 		)
 		(property "Description" "Unpolarized capacitor, small symbol"
-			(at 162.56 67.31 0)
-			(effects
-				(font
+			(at 167.64 67.31 0)
+			(effects
+				(font

Commit message: changement schéma
Parts:
- renumbered J602 to J601
Changed lines of the file:
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@@
+		(dnp no)
+		(fields_autoplaced yes)
+		(property "Reference" "#PWR0605"
+			(at 166.37 71.12 0)
+			(effects
+				(font
+					(size 1.27 1.27)
+				)
+				(hide yes)
+			)
+		)
+		(property "Value" "+3.3V"
+			(at 158.75 71.1199 90)
+			(effects
+				(font
+					(size 1.27 1.27)
+				)
+				(justify left)
+			)
+		)
+		(property "Footprint" ""
+			(at 162.56 71.12 0)
+			(effects
+				(font
+					(size 1.27 1.27)
+				)
+				(hide yes)
+			)
+		)
+		(property "Datasheet" ""
+			(at 162.56 71.12 0)
+			(effects
+				(font
+					(size 1.27 1.27)
+				)
+				(hide yes)
+			)
+		)
+		(property "Description" "Power symbol creates a global label with name \"+3.3V\""
+			(at 162.56 71.12 0)
+			(effects
+				(font
+					(size 1.27 1.27)
+				)
+				(hide yes)
+			)
+		)
+		(pin "1"
+		)
+		(instances
+			(project "Projet_torero"
+				(path "/04e1eb47-a2c4-462b-bef7-377d9515a2c0/dd27f41c-7d47-40cd-8124-f9caabbde9e3/0f1c410a-6af4-4b35-8e5a-494d8e966509"
+					(reference "#PWR0605")
+					(unit 1)
+				)
+				(path "/04e1eb47-a2c4-462b-bef7-377d9515a2c0/dd27f41c-7d47-40cd-8124-f9caabbde9e3/1155aff2-0474-4d72-be32-a9f851f4a9bf"
+					(reference "#PWR0705")
+					(unit 1)
+				)
+			)
+		)
+	)
+	(symbol
+		(lib_id "Device:C_Small")
+		(at 167.64 67.31 0)
+		(unit 1)
+		(exclude_from_sim no)
+		(in_bom yes)
+		(on_board yes)
+		(dnp no)
+		(property "Reference" "C603"
+			(at 163.576 67.564 90)
+			(effects
+				(font
+					(size 1.27 1.27)
+				)
+			)
+		)
+		(property "Value" "1u"
+			(at 161.036 67.564 90)
+			(effects
+				(font
+					(size 1.27 1.27)
+				)
+			)
+		)
+		(property "Footprint" ""
+			(at 167.64 67.31 0)
+			(effects
+				(font
+					(size 1.27 1.27)
+				)
+				(hide yes)
+			)
+		)
+		(property "Datasheet" "~"
+			(at 167.64 67.31 0)
+			(effects
+				(font
+					(size 1.27 1.27)
+				)
+				(hide yes)
+			)
+		)
+		(property "Description" "Unpolarized capacitor, small symbol"
+			(at 167.64 67.31 0)
+			(effects
+				(font
+					(size 1.27 1.27)
+				)
+				(hide yes)
+			)
+		)
+		(pin "1"
+		)
+		(pin "2"
+		)
+		(instances
+			(project "Projet_torero"
+				(path "/04e1eb47-a2c4-462b-bef7-377d9515a2c0/dd27f41c-7d47-40cd-8124-f9caabbde9e3/0f1c410a-6af4-4b35-8e5a-494d8e966509"
+					(reference "C603")
+					(unit 1)
+				)
+				(path "/04e1eb47-a2c4-462b-bef7-377d9515a2c0/dd27f41c-7d47-40cd-8124-f9caabbde9e3/1155aff2-0474-4d72-be32-a9f851f4a9bf"
+					(reference "C703")
+					(unit 1)
+				)
+			)
+		)
+	)
+	(symbol
+		(lib_id "power:GND")
+		(at 124.46 45.72 0)
+		(unit 1)
+		(exclude_from_sim no)
+		(in_bom yes)
+		(on_board yes)
 		(dnp no)
 		(fields_autoplaced yes)
 		(property "Reference" "#PWR0601"
-			(at 166.37 71.12 0)
-			(effects
-				(font
-					(size 1.27 1.27)
-				)
-				(hide yes)
-			)
-		)
-		(property "Value" "+3.3V"
-			(at 158.75 71.1199 90)
-			(effects
-				(font
-					(size 1.27 1.27)
-				)
-				(justify left)
-			)
-		)
-		(property "Footprint" ""
-			(at 162.56 71.12 0)
-			(effects
-				(font
-					(size 1.27 1.27)
-				)
-				(hide yes)
-			)
-		)
-		(property "Datasheet" ""
-			(at 162.56 71.12 0)
-			(effects
-				(font
-					(size 1.27 1.27)
-				)
-				(hide yes)
-			)
-		)
-		(property "Description" "Power symbol creates a global label with name \"+3.3V\""
-			(at 162.56 71.12 0)
-			(effects
-				(font
-					(size 1.27 1.27)
-				)
-				(hide yes)
-			)
-		)
-		(pin "1"
-		)
-		(instances
-			(project "Projet_torero"
-				(path "/04e1eb47-a2c4-462b-bef7-377d9515a2c0/dd27f41c-7d47-40cd-8124-f9caabbde9e3/0f1c410a-6af4-4b35-8e5a-494d8e966509"
-					(reference "#PWR0601")
-					(unit 1)
-				)
-				(path "/04e1eb47-a2c4-462b-bef7-377d9515a2c0/dd27f41c-7d47-40cd-8124-f9caabbde9e3/1155aff2-0474-4d72-be32-a9f851f4a9bf"
-					(reference "#PWR0701")
-					(unit 1)
-				)
-			)
-		)
-	)
-	(symbol
-		(lib_id "Device:C_Small")
-		(at 167.64 67.31 0)
-		(unit 1)
-		(exclude_from_sim no)
-		(in_bom yes)
-		(on_board yes)
-		(dnp no)
-		(property "Reference" "C603"
-			(at 163.576 67.564 90)
-			(effects
-				(font
-					(size 1.27 1.27)
-				)
-			)
-		)
-		(property "Value" "1u"
-			(at 161.036 67.564 90)
-			(effects
-				(font
-					(size 1.27 1.27)
-				)
-			)
-		)
-		(property "Footprint" ""
-			(at 167.64 67.31 0)
-			(effects
-				(font
-					(size 1.27 1.27)
-				)
-				(hide yes)
-			)
-		)
-		(property "Datasheet" "~"
-			(at 167.64 67.31 0)
-			(effects
-				(font
-					(size 1.27 1.27)
-				)
-				(hide yes)
-			)
-		)
-		(property "Description" "Unpolarized capacitor, small symbol"
-			(at 167.64 67.31 0)
-			(effects
-				(font
-					(size 1.27 1.27)
-				)
-				(hide yes)
-			)
-		)
-		(pin "1"
-		)
-		(pin "2"
-		)
-		(instances
-			(project "Projet_torero"
-				(path "/04e1eb47-a2c4-462b-bef7-377d9515a2c0/dd27f41c-7d47-40cd-8124-f9caabbde9e3/0f1c410a-6af4-4b35-8e5a-494d8e966509"
-					(reference "C603")
-					(unit 1)
-				)
-				(path "/04e1eb47-a2c4-462b-bef7-377d9515a2c0/dd27f41c-7d47-40cd-8124-f9caabbde9e3/1155aff2-0474-4d72-be32-a9f851f4a9bf"
-					(reference "C703")
-					(unit 1)
-				)
-			)
-		)
-	)
-	(symbol
-		(lib_id "power:GND")
-		(at 124.46 45.72 0)
-		(unit 1)
-		(exclude_from_sim no)
-		(in_bom yes)
-		(on_board yes)
-		(dnp no)
-		(fields_autoplaced yes)
-		(property "Reference" "#PWR0603"
 			(at 124.46 52.07 0)
 			(effects
@@
 			(project "Projet_torero"
 				(path "/04e1eb47-a2c4-462b-bef7-377d9515a2c0/dd27f41c-7d47-40cd-8124-f9caabbde9e3/0f1c410a-6af4-4b35-8e5a-494d8e966509"
-					(reference "#PWR0603")
-					(unit 1)
-				)
-				(path "/04e1eb47-a2c4-462b-bef7-377d9515a2c0/dd27f41c-7d47-40cd-8124-f9caabbde9e3/1155aff2-0474-4d72-be32-a9f851f4a9bf"
-					(reference "#PWR0703")
+					(reference "#PWR0601")
+					(unit 1)
+				)
+				(path "/04e1eb47-a2c4-462b-bef7-377d9515a2c0/dd27f41c-7d47-40cd-8124-f9caabbde9e3/1155aff2-0474-4d72-be32-a9f851f4a9bf"
+					(reference "#PWR0701")
 					(unit 1)
 				)
@@
 		(dnp no)
 		(fields_autoplaced yes)
-		(property "Reference" "J602"
+		(property "Reference" "J601"
 			(at 193.04 66.0399 0)
 			(effects
@@
 			(project ""
 				(path "/04e1eb47-a2c4-462b-bef7-377d9515a2c0/dd27f41c-7d47-40cd-8124-f9caabbde9e3/0f1c410a-6af4-4b35-8e5a-494d8e966509"
-					(reference "J602")
-					(unit 1)
-				)
-				(path "/04e1eb47-a2c4-462b-bef7-377d9515a2c0/dd27f41c-7d47-40cd-8124-f9caabbde9e3/1155aff2-0474-4d72-be32-a9f851f4a9bf"
-					(reference "J702")
+					(reference "J601")
+					(unit 1)
+				)
+				(path "/04e1eb47-a2c4-462b-bef7-377d9515a2c0/dd27f41c-7d47-40cd-8124-f9caabbde9e3/1155aff2-0474-4d72-be32-a9f851f4a9bf"
+					(reference "J701")
 					(unit 1)
 				)
@@
 		(dnp no)
 		(fields_autoplaced yes)
-		(property "Reference" "#PWR0604"
+		(property "Reference" "#PWR0602"
 			(at 139.7 77.47 0)
 			(effects
@@
 			(project "Projet_torero"
 				(path "/04e1eb47-a2c4-462b-bef7-377d9515a2c0/dd27f41c-7d47-40cd-8124-f9caabbde9e3/0f1c410a-6af4-4b35-8e5a-494d8e966509"
-					(reference "#PWR0604")
-					(unit 1)
-				)
-				(path "/04e1eb47-a2c4-462b-bef7-377d9515a2c0/dd27f41c-7d47-40cd-8124-f9caabbde9e3/1155aff2-0474-4d72-be32-a9f851f4a9bf"
-					(reference "#PWR0704")
+					(reference "#PWR0602")
+					(unit 1)
+				)
+				(path "/04e1eb47-a2c4-462b-bef7-377d9515a2c0/dd27f41c-7d47-40cd-8124-f9caabbde9e3/1155aff2-0474-4d72-be32-a9f851f4a9bf"
+					(reference "#PWR0702")
 					(unit 1)
 				)
@@
 		(dnp no)
 		(fields_autoplaced yes)
-		(property "Reference" "#PWR0605"
+		(property "Reference" "#PWR0603"
 			(at 152.4 52.07 0)
 			(effects
@@
 			(project "Projet_torero"
 				(path "/04e1eb47-a2c4-462b-bef7-377d9515a2c0/dd27f41c-7d47-40cd-8124-f9caabbde9e3/0f1c410a-6af4-4b35-8e5a-494d8e966509"
-					(reference "#PWR0605")
-					(unit 1)
-				)
-				(path "/04e1eb47-a2c4-462b-bef7-377d9515a2c0/dd27f41c-7d47-40cd-8124-f9caabbde9e3/1155aff2-0474-4d72-be32-a9f851f4a9bf"
-					(reference "#PWR0705")
+					(reference "#PWR0603")
+					(unit 1)
+				)
+				(path "/04e1eb47-a2c4-462b-bef7-377d9515a2c0/dd27f41c-7d47-40cd-8124-f9caabbde9e3/1155aff2-0474-4d72-be32-a9f851f4a9bf"
+					(reference "#PWR0703")
 					(unit 1)
 				)
@@
 		(dnp no)
 		(fields_autoplaced yes)
-		(property "Reference" "#PWR0602"
+		(property "Reference" "#PWR0604"
 			(at 156.21 63.5 0)
 			(effects
@@
 			(project "Projet_torero"
 				(path "/04e1eb47-a2c4-462b-bef7-377d9515a2c0/dd27f41c-7d47-40cd-8124-f9caabbde9e3/0f1c410a-6af4-4b35-8e5a-494d8e966509"
-					(reference "#PWR0602")
-					(unit 1)
-				)
-				(path "/04e1eb47-a2c4-462b-bef7-377d9515a2c0/dd27f41c-7d47-40cd-8124-f9caabbde9e3/1155aff2-0474-4d72-be32-a9f851f4a9bf"
-					(reference "#PWR0702")
-					(unit 1)
-				)
+					(reference "#PWR0604")
+					(unit 1)
+				)
+				(path "/04e1eb47-a2c4-462b-bef7-377d9515a2c0/dd27f41c-7d47-40cd-8124-f9caabbde9e3/1155aff2-0474-4d72-be32-a9f851f4a9bf"
+					(reference "#PWR0704")
+					(unit 1)
+				)

Commit message: modif placement composant
Parts:
- C601, C602, C603: footprint (none) -> Capacitor_SMD:C_0603_1608Metric
- J601: footprint (none) -> Connector_JST:JST_XH_S6B-XH-A_1x06_P2.50mm_Horizontal
Changed lines of the file:
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@@
 			)
 		)
-		(property "Footprint" ""
+		(property "Footprint" "Capacitor_SMD:C_0603_1608Metric"
 			(at 167.64 67.31 0)
 			(effects
@@
 			)
 		)
-		(property "Footprint" ""
+		(property "Footprint" "Connector_JST:JST_XH_S6B-XH-A_1x06_P2.50mm_Horizontal"
 			(at 190.5 66.04 0)
 			(effects
@@
 			)
 		)
-		(property "Footprint" ""
+		(property "Footprint" "Capacitor_SMD:C_0603_1608Metric"
 			(at 130.81 45.72 0)
 			(effects
@@
 			)
 		)
-		(property "Footprint" ""
+		(property "Footprint" "Capacitor_SMD:C_0603_1608Metric"
 			(at 149.86 45.72 0)
 			(effects

Commit message: Placement des composant "terminé"
Connections:
- net V7.2 renamed 7.2V
Changed lines of the file:
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@@
 		)
 	)
-	(global_label "V7.2"
+	(global_label "7.2V"
 		(shape input)
 		(at 142.24 35.56 90)

Commit message: Correction du PCB pour prof
Changed lines of the file:
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@@
+	(wire
+		(pts
+			(xy 181.61 68.58) (xy 185.42 68.58)
+		)
+		(stroke
+			(width 0)
+			(type default)
+		)
+	)
 	(wire
 		(pts
@@
 	(wire
 		(pts
+			(xy 181.61 66.04) (xy 185.42 66.04)
+		)
+		(stroke
+			(width 0)
+			(type default)
+		)
+	)
+	(wire
+		(pts
 			(xy 119.38 63.5) (xy 129.54 63.5)
 		)
@@
 	(wire
 		(pts
-			(xy 123.19 80.01) (xy 123.19 66.04)
-		)
-		(stroke
-			(width 0)
-			(type default)
-		)
-	)
-	(wire
-		(pts
 			(xy 124.46 45.72) (xy 128.27 45.72)
 		)
@@
 	(wire
 		(pts
-			(xy 119.38 80.01) (xy 119.38 63.5)
-		)
-		(stroke
-			(width 0)
-			(type default)
-		)
-	)
-	(wire
-		(pts
 			(xy 167.64 63.5) (xy 167.64 64.77)
 		)
@@
 		(pts
 			(xy 167.64 63.5) (xy 185.42 63.5)
+		)
+		(stroke
+			(width 0)
+			(type default)
+		)
+	)
+	(wire
+		(pts
+			(xy 123.19 66.04) (xy 123.19 80.01)
+		)
+		(stroke
+			(width 0)
+			(type default)
+		)
+	)
+	(wire
+		(pts
+			(xy 119.38 63.5) (xy 119.38 80.01)
 		)
 		(stroke
@@
 	(hierarchical_label "EncodeurA"
 		(shape input)
-		(at 185.42 66.04 180)
+		(at 181.61 66.04 180)
 		(fields_autoplaced yes)
 		(effects
@@
 	(hierarchical_label "EncodeurB"
 		(shape input)
-		(at 185.42 68.58 180)
+		(at 181.61 68.58 180)
 		(fields_autoplaced yes)
 		(effects

Commit message: Correction suggestion prof
Connections:
- net Commande moteur: now reaches J601.1 (Pin_1)
- net Commande moteur: now also U601.7 (OUT2); no longer U601.1 (OUT1)
- net Connecteur Moteur: now reaches J601.6 (Pin_6)
- net Connecteur Moteur: now also U601.1 (OUT1); no longer U601.7 (OUT2)
Other:
- note removed: "Connecteur moteur"
Changed lines of the file:
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@@
+	(wire
+		(pts
+			(xy 149.86 66.04) (xy 154.94 66.04)
+		)
+		(stroke
+			(width 0)
+			(type default)
+		)
+	)
 	(wire
 		(pts
@@
 	(wire
 		(pts
+			(xy 158.75 73.66) (xy 185.42 73.66)
+		)
+		(stroke
+			(width 0)
+			(type default)
+		)
+	)
+	(wire
+		(pts
 			(xy 181.61 68.58) (xy 185.42 68.58)
 		)
@@
 	(wire
 		(pts
-			(xy 149.86 60.96) (xy 185.42 60.96)
+			(xy 154.94 60.96) (xy 185.42 60.96)
 		)
 		(stroke
@@
 	(wire
 		(pts
+			(xy 210.82 55.88) (xy 210.82 81.28)
+		)
+		(stroke
+			(width 0)
+			(type default)
+		)
+	)
+	(wire
+		(pts
 			(xy 162.56 69.85) (xy 162.56 71.12)
 		)
@@
 	(wire
 		(pts
+			(xy 210.82 81.28) (xy 158.75 81.28)
+		)
+		(stroke
+			(width 0)
+			(type default)
+		)
+	)
+	(wire
+		(pts
+			(xy 153.67 55.88) (xy 210.82 55.88)
+		)
+		(stroke
+			(width 0)
+			(type default)
+		)
+	)
+	(wire
+		(pts
+			(xy 154.94 60.96) (xy 154.94 66.04)
+		)
+		(stroke
+			(width 0)
+			(type default)
+		)
+	)
+	(wire
+		(pts
+			(xy 153.67 55.88) (xy 153.67 60.96)
+		)
+		(stroke
+			(width 0)
+			(type default)
+		)
+	)
+	(wire
+		(pts
+			(xy 158.75 81.28) (xy 158.75 73.66)
+		)
+		(stroke
+			(width 0)
+			(type default)
+		)
+	)
+	(wire
+		(pts
 			(xy 123.19 66.04) (xy 129.54 66.04)
 		)
@@
 	(wire
 		(pts
-			(xy 149.86 73.66) (xy 149.86 66.04)
+			(xy 149.86 60.96) (xy 153.67 60.96)
 		)
 		(stroke
@@
 	(wire
 		(pts
-			(xy 149.86 73.66) (xy 185.42 73.66)
-		)
-		(stroke
-			(width 0)
-			(type default)
-		)
-	)
-	(wire
-		(pts
 			(xy 167.64 63.5) (xy 185.42 63.5)
 		)
@@
 		)
 	)
-	(text "Connecteur moteur"
-		(exclude_from_sim no)
-		(at 165.354 59.944 0)
+	(label "Connecteur Moteur"
+		(at 154.94 55.88 0)
+		(fields_autoplaced yes)
 		(effects
 			(font
 				(size 1.27 1.27)
 			)
+			(justify left bottom)
+		)
+	)
+	(label "Commande moteur"
+		(at 168.91 60.96 0)
+		(fields_autoplaced yes)
+		(effects
+			(font
+				(size 1.27 1.27)
+			)
+			(justify left bottom)
 		)
 	)
@@
 		(on_board yes)
 		(dnp no)
-		(fields_autoplaced yes)
 		(property "Reference" "#PWR0605"
 			(at 166.37 71.12 0)
@@
 		)
 		(property "Value" "+3.3V"
-			(at 158.75 71.1199 90)
+			(at 162.052 69.342 90)
 			(effects
 				(font
@@
 		(on_board yes)
 		(dnp no)
-		(fields_autoplaced yes)
 		(property "Reference" "U601"
 			(at 141.8941 71.12 0)
@@
 		)
 		(property "Value" "ZXBM5210-SP"
-			(at 141.8941 73.66 0)
+			(at 141.986 74.676 0)
 			(effects
 				(font
@@
 		(on_board yes)
 		(dnp no)
-		(fields_autoplaced yes)
 		(property "Reference" "#PWR0604"
 			(at 156.21 63.5 0)
@@
 		)
 		(property "Value" "GND"
-			(at 158.75 63.4999 90)
-			(effects
-				(font
+			(at 160.02 65.532 90)
+			(effects
+				(font
