File: PCB/Projet_torero/Moteur.kicad_sch (KiCad schematic)
At the start: 5 parts, among them J601 Conn_01x06, U601 ZXBM5210-SP

Commit message: Confirmation PCB
Il manque juste a finir le texte et mettre les logos de l'ENSEA et du groupe TORERO
Parts:
- added TP1, TP3: TestPoint, TestPoint:TestPoint_Pad_D1.5mm, symbol Connector:TestPoint
Connections:
- net FWD_MOT: now also TP1.1
- net REV_MOT: now also TP3.1
Changed lines of the file:
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@@
 	(paper "A4")
+	(junction
+		(at 119.38 71.12)
+		(diameter 0)
+		(color 0 0 0 0)
+	)
 	(junction
 		(at 162.56 71.12)
@@
 	)
 	(junction
+		(at 123.19 71.12)
+		(diameter 0)
+		(color 0 0 0 0)
+	)
+	(junction
 		(at 142.24 39.37)
 		(diameter 0)
@@
 	(wire
 		(pts
+			(xy 123.19 71.12) (xy 123.19 80.01)
+		)
+		(stroke
+			(width 0)
+			(type default)
+		)
+	)
+	(wire
+		(pts
 			(xy 181.61 66.04) (xy 185.42 66.04)
 		)
@@
 	(wire
 		(pts
-			(xy 123.19 66.04) (xy 123.19 80.01)
-		)
-		(stroke
-			(width 0)
-			(type default)
-		)
-	)
-	(wire
-		(pts
-			(xy 119.38 63.5) (xy 119.38 80.01)
+			(xy 123.19 66.04) (xy 123.19 71.12)
+		)
+		(stroke
+			(width 0)
+			(type default)
+		)
+	)
+	(wire
+		(pts
+			(xy 119.38 63.5) (xy 119.38 71.12)
 		)
 		(stroke
@@
 		(pts
 			(xy 167.64 69.85) (xy 162.56 69.85)
+		)
+		(stroke
+			(width 0)
+			(type default)
+		)
+	)
+	(wire
+		(pts
+			(xy 119.38 71.12) (xy 119.38 80.01)
 		)
 		(stroke
@@
 	)
 	(symbol
+		(lib_id "Connector:TestPoint")
+		(at 123.19 71.12 270)
+		(unit 1)
+		(exclude_from_sim no)
+		(in_bom yes)
+		(on_board yes)
+		(dnp no)
+		(fields_autoplaced yes)
+		(property "Reference" "TP3"
+			(at 128.27 69.8499 90)
+			(effects
+				(font
+					(size 1.27 1.27)
+				)
+				(justify left)
+			)
+		)
+		(property "Value" "TestPoint"
+			(at 128.27 72.3899 90)
+			(effects
+				(font
+					(size 1.27 1.27)
+				)
+				(justify left)
+			)
+		)
+		(property "Footprint" "TestPoint:TestPoint_Pad_D1.5mm"
+			(at 123.19 76.2 0)
+			(effects
+				(font
+					(size 1.27 1.27)
+				)
+				(hide yes)
+			)
+		)
+		(property "Datasheet" "~"
+			(at 123.19 76.2 0)
+			(effects
+				(font
+					(size 1.27 1.27)
+				)
+				(hide yes)
+			)
+		)
+		(property "Description" "test point"
+			(at 123.19 71.12 0)
+			(effects
+				(font
+					(size 1.27 1.27)
+				)
+				(hide yes)
+			)
+		)
+		(pin "1"
+		)
+		(instances
+			(project "Projet_torero"
+				(path "/04e1eb47-a2c4-462b-bef7-377d9515a2c0/dd27f41c-7d47-40cd-8124-f9caabbde9e3/0f1c410a-6af4-4b35-8e5a-494d8e966509"
+					(reference "TP3")
+					(unit 1)
+				)
+				(path "/04e1eb47-a2c4-462b-bef7-377d9515a2c0/dd27f41c-7d47-40cd-8124-f9caabbde9e3/1155aff2-0474-4d72-be32-a9f851f4a9bf"
+					(reference "TP4")
+					(unit 1)
+				)
+			)
+		)
+	)
+	(symbol
 		(lib_id "power:GND")
 		(at 124.46 45.72 0)
@@
 					(unit 1)
 				)
+			)
+		)
+	)
+	(symbol
+		(lib_id "Connector:TestPoint")
+		(at 119.38 71.12 90)
+		(unit 1)
+		(exclude_from_sim no)
+		(in_bom yes)
+		(on_board yes)
+		(dnp no)
+		(fields_autoplaced yes)
+		(property "Reference" "TP1"
+			(at 116.078 66.04 90)
+			(effects
+				(font
+					(size 1.27 1.27)
+				)
+			)
+		)
+		(property "Value" "TestPoint"
+			(at 116.078 68.58 90)
+			(effects
+				(font
+					(size 1.27 1.27)
+				)
+			)
+		)
+		(property "Footprint" "TestPoint:TestPoint_Pad_D1.5mm"
+			(at 119.38 66.04 0)
+			(effects
+				(font
+					(size 1.27 1.27)
+				)
+				(hide yes)
+			)
+		)
+		(property "Datasheet" "~"
+			(at 119.38 66.04 0)
+			(effects
+				(font
+					(size 1.27 1.27)
+				)
+				(hide yes)
+			)
+		)
+		(property "Description" "test point"
+			(at 119.38 71.12 0)
+			(effects
+				(font
+					(size 1.27 1.27)
+				)
+				(hide yes)
+			)
+		)
+		(pin "1"
+		)
+		(instances
+			(project ""
+				(path "/04e1eb47-a2c4-462b-bef7-377d9515a2c0/dd27f41c-7d47-40cd-8124-f9caabbde9e3/0f1c410a-6af4-4b35-8e5a-494d8e966509"
+					(reference "TP1")
+					(unit 1)
+				)
+				(path "/04e1eb47-a2c4-462b-bef7-377d9515a2c0/dd27f41c-7d47-40cd-8124-f9caabbde9e3/1155aff2-0474-4d72-be32-a9f851f4a9bf"
+					(reference "TP2")
+					(unit 1)
+				)
